File: AudioFront.kicad_sch (KiCad schematic)
At the start: 10 parts, among them J1 NJ2FD-V, U5 TL072, U6 TLV9062

Commit message: test git
Parts:
- added R6: TEST, symbol Device:R
Changed lines of the file:
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@@
+	)
+	(symbol
+		(lib_id "Device:R")
+		(at 115.57 105.41 0)
+		(unit 1)
+		(exclude_from_sim no)
+		(in_bom yes)
+		(on_board yes)
+		(dnp no)
+		(fields_autoplaced yes)
+		(property "Reference" "R6"
+			(at 118.11 104.1399 0)
+			(effects
+				(font
+					(size 1.27 1.27)
+				)
+				(justify left)
+			)
+		)
+		(property "Value" "TEST"
+			(at 118.11 106.6799 0)
+			(effects
+				(font
+					(size 1.27 1.27)
+				)
+				(justify left)
+			)
+		)
+		(property "Footprint" ""
+			(at 113.792 105.41 90)
+			(effects
+				(font
+					(size 1.27 1.27)
+				)
+				(hide yes)
+			)
+		)
+		(property "Datasheet" "~"
+			(at 115.57 105.41 0)
+			(effects
+				(font
+					(size 1.27 1.27)
+				)
+				(hide yes)
+			)
+		)
+		(property "Description" "Resistor"
+			(at 115.57 105.41 0)
+			(effects
+				(font
+					(size 1.27 1.27)
+				)
+				(hide yes)
+			)
+		)
+		(pin "2"
+		)
+		(pin "1"
+		)
+		(instances
+			(project "DSPboard"
+				(path "/ee8026cd-c8f1-4ab8-b3ed-795cda0e45f2/b0d28cc3-ef70-4b40-ae3e-ad3f3c6b0382"
+					(reference "R6")
+					(unit 1)
+				)
+			)
+		)
 	)
 	(symbol
